File: Board/Can_Gauge/Can_Gauge.kicad_sch (KiCad schematic)
At the start: 33 parts, among them J1 FTDI-Port, J2 CAN, J3 LED 12V, J4 12V, J5 GND, M1 Stepper_Motor, U1 ATMEGA328P-AU, U2 MCP2515-xST, U3 MCP2551-I-SN, U4 L78L05_SOT89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

Commit message: Board adjustments
Parts:
- D7, D8, D9: LCSC C2827311 -> C2843869

Commit message: Gauge faces; Init move; restructure Board
Parts:
- removed J3: LED 12V, Connector_PinHeader_2.54mm:PinHeader_1x01_P2.54mm_Vertical, symbol Connector:Conn_01x01_Pin
- added J6: 12V_LED_Bridge, Connector_PinHeader_2.54mm:PinHeader_1x02_P2.54mm_Vertical, symbol Connector:Conn_01x02_Pin
- added J7: SPI-Port, Connector_PinHeader_1.00mm:PinHeader_2x03_P1.00mm_Vertical, symbol Connector:Conn_01x06_Pin
Connections:
- net +12V: now also J6.1 (Pin_1)
- net +5V: now also J7.4 (Pin_4)
- net 12V_LED: now also J6.2 (Pin_2)
- net DTR: now also J7.2 (Pin_2)
- net GND: now also J7.6 (Pin_6)
- net SPI_MISO: now reaches U1.15 (PB3), U2.16 (SI)
- net SPI_MISO: now also J7.5 (Pin_5)
- net SPI_MOSI: now reaches U1.16 (PB4), U2.17 (SO)
- net SPI_MOSI: now also J7.3 (Pin_3)
- net SPI_CLK: now reaches U1.17 (PB5), U2.14 (SCK)
- net SPI_CLK: now also J7.1 (Pin_1)

Commit message: Board: Add protection Diode
Parts:
- added D10: D, Diode_SMD:D_SOD-123F, symbol Device:D
- J7: footprint Connector_PinHeader_1.00mm:PinHeader_2x03_P1.00mm_Vertical -> Connector_PinHeader_1.27mm:PinHeader_2x03_P1.27mm_Vertical
Connections:
- net +12V: now also D10.2 (A); no longer U4.3 (IN)
- net DTR: no longer J7.2 (Pin_2)
- net Reset: now reaches C3.2, R2.1, U1.29 (PC6)
- net Reset: now also J7.2 (Pin_2)
- new net: D10.1 (K), U4.3 (IN)
Other:
- moved on the sheet: J1
